File: chime.kicad_pcb (KiCad board)
At the start: 2 copper layers, 231.1 x 134.6 mm, 20 parts, among them J1 Conn_01x02, J2 Conn_01x10, J3 Conn_01x04, K1 G5LE-1, U1 L7805, U10 NJM4558, U11 NJM4558, U2 4050, U3 4042, U4 4081, U5 4011, U6 4011, U7 4024, U8 40245, U9 NJM4558

Commit message: resistors
Parts:
- added C16: C, Capacitor_THT:C_Disc_D10.0mm_W2.5mm_P5.00mm, F.Cu at (141.1, 162.6)
- added C25: C, Capacitor_THT:C_Disc_D10.0mm_W2.5mm_P5.00mm, F.Cu at (90.2, 50.7)
- added C36: C, Capacitor_THT:C_Disc_D10.0mm_W2.5mm_P5.00mm, F.Cu at (167.7, 52.1)
- added C4: 100u, Capacitor_THT:CP_Radial_D8.0mm_P3.50mm, F.Cu at (207.3, 144.8)
- added C5: C, Capacitor_THT:C_Disc_D10.0mm_W2.5mm_P5.00mm, F.Cu at (210.9, 134.6)
- added D1: D_Bridge_+-AA, Diode_THT:Diode_Bridge_Vishay_KBL, F.Cu at (231.1, 105.4)
- added D2: D, Diode_THT:D_A-405_P10.16mm_Horizontal, F.Cu at (221.0, 129.5)
- added D3: D, Diode_THT:D_A-405_P10.16mm_Horizontal, F.Cu at (208.3, 61.0)
- added D4: D, Diode_THT:D_A-405_P10.16mm_Horizontal, F.Cu at (157.5, 113.0)
- added D5: D, Diode_THT:D_A-405_P10.16mm_Horizontal, F.Cu at (157.5, 129.5)
- added D6: D, Diode_THT:D_A-405_P10.16mm_Horizontal, F.Cu at (161.3, 113.0)
- added D7: D, Diode_THT:D_A-405_P10.16mm_Horizontal, F.Cu at (222.2, 78.7)
- added DA8: D, Diode_THT:D_A-405_P10.16mm_Horizontal, F.Cu at (55.9, 157.5)
- added DB8: D, Diode_THT:D_A-405_P10.16mm_Horizontal, F.Cu at (55.9, 144.8)
- added DC8: D, Diode_THT:D_A-405_P10.16mm_Horizontal, F.Cu at (52.1, 134.8)
- added DD8: D, Diode_THT:D_A-405_P10.16mm_Horizontal, F.Cu at (55.9, 127.0)
- added H1: MountingHole, MountingHole:MountingHole_3.2mm_M3, F.Cu at (241.3, 68.6)
- added H2: MountingHole, MountingHole:MountingHole_3.2mm_M3, F.Cu at (241.3, 160.0)
- added H3: MountingHole, MountingHole:MountingHole_3.2mm_M3, F.Cu at (156.2, 67.3)
- added H4: MountingHole, MountingHole:MountingHole_3.2mm_M3, F.Cu at (156.2, 157.5)
- added H5: MountingHole, MountingHole:MountingHole_3.2mm_M3, F.Cu at (41.9, 157.5)
- added H6: MountingHole, MountingHole:MountingHole_3.2mm_M3, F.Cu at (31.8, 166.4)
- added R1: ~, Resistor_THT:R_Axial_DIN0207_L6.3mm_D2.5mm_P10.16mm_Horizontal, F.Cu at (238.8, 128.3)
- added R11: ~, Resistor_THT:R_Axial_DIN0207_L6.3mm_D2.5mm_P10.16mm_Horizontal, F.Cu at (194.3, 151.1)
- added R12: ~, Resistor_THT:R_Axial_DIN0207_L6.3mm_D2.5mm_P10.16mm_Horizontal, F.Cu at (161.3, 63.5)
- added R13: ~, Resistor_THT:R_Axial_DIN0207_L6.3mm_D2.5mm_P10.16mm_Horizontal, F.Cu at (138.4, 80.0)
- added R14: ~, Resistor_THT:R_Axial_DIN0207_L6.3mm_D2.5mm_P10.16mm_Horizontal, F.Cu at (147.3, 127.0)
- added R15: ~, Resistor_THT:R_Axial_DIN0207_L6.3mm_D2.5mm_P10.16mm_Horizontal, F.Cu at (157.5, 94.0)
- added R16: ~, Resistor_THT:R_Axial_DIN0207_L6.3mm_D2.5mm_P10.16mm_Horizontal, F.Cu at (161.3, 94.0)
- added R2: 39R 2W, Resistor_THT:R_Axial_DIN0516_L15.5mm_D5.0mm_P20.32mm_Horizontal, F.Cu at (243.8, 139.7)
- added R23: 1k, Resistor_THT:R_Axial_DIN0207_L6.3mm_D2.5mm_P10.16mm_Horizontal, F.Cu at (82.5, 167.6)
- added R28: 470k, Resistor_THT:R_Axial_DIN0207_L6.3mm_D2.5mm_P10.16mm_Horizontal, F.Cu at (109.2, 53.3)
- added R3: 1k, Resistor_THT:R_Axial_DIN0207_L6.3mm_D2.5mm_P10.16mm_Horizontal, F.Cu at (223.5, 129.5)
- added R31: 3.3k, Resistor_THT:R_Axial_DIN0207_L6.3mm_D2.5mm_P10.16mm_Horizontal, F.Cu at (97.8, 68.6)
- added R34: 3.3k, Resistor_THT:R_Axial_DIN0207_L6.3mm_D2.5mm_P10.16mm_Horizontal, F.Cu at (110.5, 74.9)
- added R38: 2.2k, Resistor_THT:R_Axial_DIN0207_L6.3mm_D2.5mm_P10.16mm_Horizontal, F.Cu at (94.0, 158.8)
- added R39: 1k, Resistor_THT:R_Axial_DIN0207_L6.3mm_D2.5mm_P10.16mm_Horizontal, F.Cu at (104.1, 163.8)
- added R4: 1k, Resistor_THT:R_Axial_DIN0207_L6.3mm_D2.5mm_P10.16mm_Horizontal, F.Cu at (223.5, 133.3)
- added R40: 2.2k, Resistor_THT:R_Axial_DIN0207_L6.3mm_D2.5mm_P10.16mm_Horizontal, F.Cu at (94.0, 154.9)
- added R46: 3.3k, Resistor_THT:R_Axial_DIN0207_L6.3mm_D2.5mm_P10.16mm_Horizontal, F.Cu at (127.0, 83.8)
- added R5: ~, Resistor_THT:R_Axial_DIN0207_L6.3mm_D2.5mm_P10.16mm_Horizontal, F.Cu at (240.0, 101.6)
- added R51: 470, Resistor_THT:R_Axial_DIN0207_L6.3mm_D2.5mm_P10.16mm_Horizontal, F.Cu at (43.2, 53.3)
- added R53: 22k, Resistor_THT:R_Axial_DIN0207_L6.3mm_D2.5mm_P10.16mm_Horizontal, F.Cu at (35.6, 121.9)
- added R54: 22k, Resistor_THT:R_Axial_DIN0207_L6.3mm_D2.5mm_P10.16mm_Horizontal, F.Cu at (35.6, 116.8)
- added R55: 2.2k, Resistor_THT:R_Axial_DIN0207_L6.3mm_D2.5mm_P10.16mm_Horizontal, F.Cu at (67.3, 109.2)
- added R56: 22k, Resistor_THT:R_Axial_DIN0207_L6.3mm_D2.5mm_P10.16mm_Horizontal, F.Cu at (63.5, 109.2)
- added R58: 470k, Resistor_THT:R_Axial_DIN0207_L6.3mm_D2.5mm_P10.16mm_Horizontal, F.Cu at (39.4, 95.2)
- added R6: ~, Resistor_THT:R_Axial_DIN0207_L6.3mm_D2.5mm_P10.16mm_Horizontal, F.Cu at (240.0, 97.8)
- added R60: 2.2k, Resistor_THT:R_Axial_DIN0207_L6.3mm_D2.5mm_P10.16mm_Horizontal, F.Cu at (39.4, 90.2)
- added R61: 470, Resistor_THT:R_Axial_DIN0207_L6.3mm_D2.5mm_P10.16mm_Horizontal, F.Cu at (34.3, 90.2)
- added R9: ~, Resistor_THT:R_Axial_DIN0207_L6.3mm_D2.5mm_P10.16mm_Horizontal, F.Cu at (174.0, 141.0)
- added RA10: 22k, Resistor_THT:R_Axial_DIN0207_L6.3mm_D2.5mm_P10.16mm_Horizontal, F.Cu at (193.0, 105.4)
- added RA7: ~, Resistor_THT:R_Axial_DIN0207_L6.3mm_D2.5mm_P10.16mm_Horizontal, F.Cu at (236.2, 88.9)
- added RA8: 470k, Resistor_THT:R_Axial_DIN0207_L6.3mm_D2.5mm_P10.16mm_Horizontal, F.Cu at (207.0, 89.6)
- added RB10: 22k, Resistor_THT:R_Axial_DIN0207_L6.3mm_D2.5mm_P10.16mm_Horizontal, F.Cu at (193.0, 110.5)
- added RB7: ~, Resistor_THT:R_Axial_DIN0207_L6.3mm_D2.5mm_P10.16mm_Horizontal, F.Cu at (236.2, 85.1)
- added RB8: 470k, Resistor_THT:R_Axial_DIN0207_L6.3mm_D2.5mm_P10.16mm_Horizontal, F.Cu at (207.0, 85.6)
- added RC10: 22k, Resistor_THT:R_Axial_DIN0207_L6.3mm_D2.5mm_P10.16mm_Horizontal, F.Cu at (193.0, 121.9)
- added RC7: ~, Resistor_THT:R_Axial_DIN0207_L6.3mm_D2.5mm_P10.16mm_Horizontal, F.Cu at (236.2, 81.3)
- added RC8: 470k, Resistor_THT:R_Axial_DIN0207_L6.3mm_D2.5mm_P10.16mm_Horizontal, F.Cu at (207.0, 81.5)
- added RD10: 22k, Resistor_THT:R_Axial_DIN0207_L6.3mm_D2.5mm_P10.16mm_Horizontal, F.Cu at (193.0, 128.3)
- added RD7: ~, Resistor_THT:R_Axial_DIN0207_L6.3mm_D2.5mm_P10.16mm_Horizontal, F.Cu at (236.2, 77.5)
- added RD8: 470k, Resistor_THT:R_Axial_DIN0207_L6.3mm_D2.5mm_P10.16mm_Horizontal, F.Cu at (207.0, 77.5)
- added RV1: 473, Potentiometer_THT:Potentiometer_Runtron_RM-065_Vertical, F.Cu at (83.9, 61.0)
- added RV2: 473, Potentiometer_THT:Potentiometer_Runtron_RM-065_Vertical, F.Cu at (43.2, 61.0)
- added RV3: 473, Potentiometer_THT:Potentiometer_Runtron_RM-065_Vertical, F.Cu at (104.2, 89.0)
- added RV4: 473, Potentiometer_THT:Potentiometer_Runtron_RM-065_Vertical, F.Cu at (122.0, 89.0)
- added SW1: AudioJack3_Ground_Switch, Connector_Audio:Jack_6.35mm_Neutrik_NMJ6HCD2_Horizontal, F.Cu at (78.7, 43.2)
- added SW2: SW_SPDT, Button_Switch_THT:SW_E-Switch_EG1224_SPDT_Angled, F.Cu at (43.7, 46.2)
- added TP6: ~, TestPoint:TestPoint_Keystone_5000-5004_Miniature, F.Cu at (91.4, 162.6)
- U8: value 40245 -> 74S472
- moved U9 1.80 mm to (110.5, 57.1)
- moved J1 1.80 mm to (245.1, 107.7)
- moved U8 1.80 mm to (113.0, 125.7)
- moved TP4 1.27 mm to (116.8, 92.7)
- moved U3 1.27 mm to (181.6, 111.8)
- moved U7 1.27 mm to (139.7, 141.0)
- moved U2 1.27 mm to (181.6, 68.6)
- moved U4 1.27 mm to (179.1, 152.4)
Connections:
- U8 pad 1: unconnected-(U8-Dir-Pad1) -> /A0
- U8 pad 10: unconnected-(U8-Vss-Pad10) -> GND
- U8 pad 11: unconnected-(U8-Pad11) -> /D4
- U8 pad 12: unconnected-(U8-Pad12) -> /D5
- U8 pad 13: unconnected-(U8-Pad13) -> /D6
- U8 pad 14: unconnected-(U8-Pad14) -> /D7
- U8 pad 16: unconnected-(U8-Pad16) -> /A5
- U8 pad 17: unconnected-(U8-Pad17) -> /A6
- U8 pad 18: unconnected-(U8-Pad18) -> /A7
- U8 pad 19: unconnected-(U8-~{G}-Pad19) -> /A8
- U8 pad 2: unconnected-(U8-Pad2) -> /A1
- U8 pad 3: unconnected-(U8-Pad3) -> /A2
- U8 pad 4: unconnected-(U8-Pad4) -> /A3
- U8 pad 5: unconnected-(U8-Pad5) -> /A4
- U8 pad 6: unconnected-(U8-Pad6) -> /D0
- U8 pad 7: unconnected-(U8-Pad7) -> /D1
- U8 pad 8: unconnected-(U8-Pad8) -> /D2
- U8 pad 9: unconnected-(U8-Pad9) -> /D3
Other:
- board text added: "SSK0035-1"

Commit message: moar parts
Parts:
- removed R5, R6: ~, Resistor_THT:R_Axial_DIN0207_L6.3mm_D2.5mm_P10.16mm_Horizontal
- added C14: C_Polarized, Capacitor_THT:CP_Radial_D5.0mm_P2.50mm, F.Cu at (156.8, 105.4)
- added C15: 47u, Capacitor_THT:CP_Radial_D5.0mm_P2.50mm, F.Cu at (163.8, 128.3)
- added C8: ~, Capacitor_THT:CP_Radial_D8.0mm_P3.50mm, F.Cu at (216.2, 144.8)
- added R17: ~, Resistor_THT:R_Axial_DIN0207_L6.3mm_D2.5mm_P10.16mm_Horizontal, F.Cu at (160.0, 99.1)
- added R18: ~, Resistor_THT:R_Axial_DIN0207_L6.3mm_D2.5mm_P10.16mm_Horizontal, F.Cu at (124.5, 156.2)
- added R19: ~, Resistor_THT:R_Axial_DIN0207_L6.3mm_D2.5mm_P10.16mm_Horizontal, F.Cu at (163.8, 123.2)
- added R20: ~, Resistor_THT:R_Axial_DIN0207_L6.3mm_D2.5mm_P10.16mm_Horizontal, F.Cu at (166.4, 165.1)
- added R27: ~, Resistor_THT:R_Axial_DIN0207_L6.3mm_D2.5mm_P10.16mm_Horizontal, F.Cu at (109.2, 49.5)
- added R29: ~, Resistor_THT:R_Axial_DIN0207_L6.3mm_D2.5mm_P10.16mm_Horizontal, F.Cu at (101.6, 68.6)
- added R30: ~, Resistor_THT:R_Axial_DIN0207_L6.3mm_D2.5mm_P10.16mm_Horizontal, F.Cu at (105.4, 68.6)
- added R32: ~, Resistor_THT:R_Axial_DIN0207_L6.3mm_D2.5mm_P10.16mm_Horizontal, F.Cu at (109.9, 80.0)
- added R33: ~, Resistor_THT:R_Axial_DIN0207_L6.3mm_D2.5mm_P10.16mm_Horizontal, F.Cu at (126.4, 67.9)
- added R35: ~, Resistor_THT:R_Axial_DIN0207_L6.3mm_D2.5mm_P10.16mm_Horizontal, F.Cu at (110.5, 71.1)
- added R36: ~, Resistor_THT:R_Axial_DIN0207_L6.3mm_D2.5mm_P10.16mm_Horizontal, F.Cu at (122.6, 67.9)
- added R37: ~, Resistor_THT:R_Axial_DIN0207_L6.3mm_D2.5mm_P10.16mm_Horizontal, F.Cu at (125.1, 46.4)
- added R41: ~, Resistor_THT:R_Axial_DIN0207_L6.3mm_D2.5mm_P10.16mm_Horizontal, F.Cu at (94.0, 150.5)
- added R42: ~, Resistor_THT:R_Axial_DIN0207_L6.3mm_D2.5mm_P10.16mm_Horizontal, F.Cu at (110.5, 157.5)
- added R45: ~, Resistor_THT:R_Axial_DIN0207_L6.3mm_D2.5mm_P10.16mm_Horizontal, F.Cu at (94.6, 68.6)
- added R47: 1k, Resistor_THT:R_Axial_DIN0207_L6.3mm_D2.5mm_P10.16mm_Horizontal, F.Cu at (86.4, 82.5)
- added R52: ~, Resistor_THT:R_Axial_DIN0207_L6.3mm_D2.5mm_P10.16mm_Horizontal, F.Cu at (35.6, 125.7)
- added R57: ~, Resistor_THT:R_Axial_DIN0207_L6.3mm_D2.5mm_P10.16mm_Horizontal, F.Cu at (35.6, 113.7)
- added R59: ~, Resistor_THT:R_Axial_DIN0207_L6.3mm_D2.5mm_P10.16mm_Horizontal, F.Cu at (39.4, 99.1)
- added RA21: ~, Resistor_THT:R_Axial_DIN0207_L6.3mm_D2.5mm_P10.16mm_Horizontal, F.Cu at (108.0, 137.2)
- added RA22: 1k, Resistor_THT:R_Axial_DIN0207_L6.3mm_D2.5mm_P10.16mm_Horizontal, F.Cu at (106.7, 132.1)
- added RA25: ~, Resistor_THT:R_Axial_DIN0207_L6.3mm_D2.5mm_P10.16mm_Horizontal, F.Cu at (45.7, 143.6)
- added RA5: ~, Resistor_THT:R_Axial_DIN0207_L6.3mm_D2.5mm_P10.16mm_Horizontal, F.Cu at (248.9, 101.0)
- added RA6: ~, Resistor_THT:R_Axial_DIN0207_L6.3mm_D2.5mm_P10.16mm_Horizontal, F.Cu at (248.9, 97.8)
- added RB21: ~, Resistor_THT:R_Axial_DIN0207_L6.3mm_D2.5mm_P10.16mm_Horizontal, F.Cu at (104.8, 137.2)
- added RB22: 1k, Resistor_THT:R_Axial_DIN0207_L6.3mm_D2.5mm_P10.16mm_Horizontal, F.Cu at (106.7, 127.0)
- added RB25: ~, Resistor_THT:R_Axial_DIN0207_L6.3mm_D2.5mm_P10.16mm_Horizontal, F.Cu at (45.7, 139.1)
- added RB5: ~, Resistor_THT:R_Axial_DIN0207_L6.3mm_D2.5mm_P10.16mm_Horizontal, F.Cu at (248.9, 94.6)
- added RB6: ~, Resistor_THT:R_Axial_DIN0207_L6.3mm_D2.5mm_P10.16mm_Horizontal, F.Cu at (248.9, 90.8)
- added RC21: ~, Resistor_THT:R_Axial_DIN0207_L6.3mm_D2.5mm_P10.16mm_Horizontal, F.Cu at (101.6, 137.2)
- added RC22: 1k, Resistor_THT:R_Axial_DIN0207_L6.3mm_D2.5mm_P10.16mm_Horizontal, F.Cu at (106.7, 121.9)
- added RC25: ~, Resistor_THT:R_Axial_DIN0207_L6.3mm_D2.5mm_P10.16mm_Horizontal, F.Cu at (45.7, 134.6)
- added RC5: ~, Resistor_THT:R_Axial_DIN0207_L6.3mm_D2.5mm_P10.16mm_Horizontal, F.Cu at (248.9, 87.6)
- added RC6: ~, Resistor_THT:R_Axial_DIN0207_L6.3mm_D2.5mm_P10.16mm_Horizontal, F.Cu at (248.9, 84.5)
- added RD21: ~, Resistor_THT:R_Axial_DIN0207_L6.3mm_D2.5mm_P10.16mm_Horizontal, F.Cu at (98.4, 137.2)
- added RD22: 1k, Resistor_THT:R_Axial_DIN0207_L6.3mm_D2.5mm_P10.16mm_Horizontal, F.Cu at (106.7, 116.8)
- added RD25: ~, Resistor_THT:R_Axial_DIN0207_L6.3mm_D2.5mm_P10.16mm_Horizontal, F.Cu at (45.7, 129.5)
- added RD5: ~, Resistor_THT:R_Axial_DIN0207_L6.3mm_D2.5mm_P10.16mm_Horizontal, F.Cu at (248.9, 80.6)
- added RD6: ~, Resistor_THT:R_Axial_DIN0207_L6.3mm_D2.5mm_P10.16mm_Horizontal, F.Cu at (248.9, 77.5)
- moved D3 1.42 mm to (207.0, 60.3)
- moved K1 1.42 mm to (213.3, 66.4)
