File: chime.kicad_sch (KiCad schematic)
At the start: 20 parts, among them J1 Conn_01x02, J2 Conn_01x10, J3 Conn_01x04, K1 G5LE-1, U1 L7805, U10 NJM4558, U11 NJM4558, U2 4050, U3 4042, U4 4081, U5 4011, U6 4011, U7 4024, U8 40245, U9 NJM4558

Commit message: resistors
Parts:
- removed U8: 40245, Package_DIP:DIP-20_W7.62mm, symbol 4xxx_IEEE:40245
- added C16, C25, C36, C5: C, Capacitor_THT:C_Disc_D10.0mm_W2.5mm_P5.00mm, symbol Device:C
- added C4: 100u, Capacitor_THT:CP_Radial_D8.0mm_P3.50mm, symbol Device:C_Polarized
- added D1: D_Bridge_+-AA, Diode_THT:Diode_Bridge_Vishay_KBL, symbol Device:D_Bridge_+-AA
- added D2, D3, D4, D5, D6, D7, DA8, DB8, DC8, DD8: D, Diode_THT:D_A-405_P10.16mm_Horizontal, symbol Device:D
- added H1, H2, H3, H4, H5, H6: MountingHole, MountingHole:MountingHole_3.2mm_M3, symbol Mechanical:MountingHole
- added R1, R11, R12, R13, R14, R15, R16, R5, R6, R9, RA7, RB7, RC7, RD7: ~, Resistor_THT:R_Axial_DIN0207_L6.3mm_D2.5mm_P10.16mm_Horizontal, symbol Device:R
- added R2: 39R 2W, Resistor_THT:R_Axial_DIN0516_L15.5mm_D5.0mm_P20.32mm_Horizontal, symbol Device:R
- added R23, R3, R39, R4: 1k, Resistor_THT:R_Axial_DIN0207_L6.3mm_D2.5mm_P10.16mm_Horizontal, symbol Device:R
- added R28, R58, RA8, RB8, RC8, RD8: 470k, Resistor_THT:R_Axial_DIN0207_L6.3mm_D2.5mm_P10.16mm_Horizontal, symbol Device:R
- added R31, R34, R46: 3.3k, Resistor_THT:R_Axial_DIN0207_L6.3mm_D2.5mm_P10.16mm_Horizontal, symbol Device:R
- added R38, R40, R55, R60: 2.2k, Resistor_THT:R_Axial_DIN0207_L6.3mm_D2.5mm_P10.16mm_Horizontal, symbol Device:R
- added R51, R61: 470, Resistor_THT:R_Axial_DIN0207_L6.3mm_D2.5mm_P10.16mm_Horizontal, symbol Device:R
- added R53, R54, R56, RA10, RB10, RC10, RD10: 22k, Resistor_THT:R_Axial_DIN0207_L6.3mm_D2.5mm_P10.16mm_Horizontal, symbol Device:R
- added RV1, RV2, RV3, RV4: 473, Potentiometer_THT:Potentiometer_Runtron_RM-065_Vertical, symbol Device:R_Potentiometer
- added SW1: AudioJack3_Ground_Switch, Connector_Audio:Jack_6.35mm_Neutrik_NMJ6HCD2_Horizontal, symbol Connector_Audio:AudioJack3_Ground_Switch
- added SW2: SW_SPDT, Button_Switch_THT:SW_E-Switch_EG1224_SPDT_Angled, symbol Switch:SW_SPDT
- added TP6: ~, TestPoint:TestPoint_Keystone_5000-5004_Miniature, symbol Connector:TestPoint
- added U8: 74S472, Package_DIP:DIP-20_W7.62mm, symbol BPROM:74S472
Connections:
- new net A0: U8.1 (A0)
- new net A1: U8.2 (A1)
- new net A2: U8.3 (A2)
- new net A3: U8.4 (A3)
- new net A4: U8.5 (A4)
- new net A5: U8.16 (A5)
- new net A6: U8.17 (A6)
- new net A7: U8.18 (A7)
- new net A8: U8.19 (A8)
- new net D0: U8.6 (Q0)
- new net D1: U8.7 (Q1)
- new net D2: U8.8 (Q2)
- new net D3: U8.9 (Q3)
- new net D4: U8.11 (Q4)
- new net D5: U8.12 (Q5)
- new net D6: U8.13 (Q6)
- new net D7: U8.14 (Q7)
- new net GND: U8.10 (GND)

Commit message: moar parts
Parts:
- removed R5, R6: ~, Resistor_THT:R_Axial_DIN0207_L6.3mm_D2.5mm_P10.16mm_Horizontal, symbol Device:R
- added C14: C_Polarized, Capacitor_THT:CP_Radial_D5.0mm_P2.50mm, symbol Device:C_Polarized
- added C15: 47u, Capacitor_THT:CP_Radial_D5.0mm_P2.50mm, symbol Device:C_Polarized
- added C8: ~, Capacitor_THT:CP_Radial_D8.0mm_P3.50mm, symbol Device:C_Polarized
- added R17, R18, R19, R20, R27, R29, R30, R32, R33, R35, R36, R37, R41, R42, R45, R52, R57, R59, RA21, RA25, RA5, RA6, RB21, RB25, RB5, RB6, RC21, RC25, RC5, RC6, RD21, RD25, RD5, RD6: ~, Resistor_THT:R_Axial_DIN0207_L6.3mm_D2.5mm_P10.16mm_Horizontal, symbol Device:R
- added R47, RA22, RB22, RC22, RD22: 1k, Resistor_THT:R_Axial_DIN0207_L6.3mm_D2.5mm_P10.16mm_Horizontal, symbol Device:R
